File: Schaltplan/CallForHelp.sch (EAGLE design)
At the start: 20 parts

Commit message: updated circuit diagram
Parts:
- removed TOGGLE_SWITCH: (no value), switch:320-916
- added SWITCH: (no value), switch:320-916
Connections:
- net N$14 renamed BATTERY_VCC
- net N$8 renamed BATTERY_GND
- removed net 5V: 5V_REGULATOR.VOUT, C1.1, C2.1, R2.2, TOGGLE_SWITCH.P, WEMOS1.5V
- removed net N$15: 5V_REGULATOR.EN, 5V_REGULATOR.VIN, C3.1, L1.1
- removed net N$16: 5V_REGULATOR.GND, 5V_REGULATOR.MODE, C2.2, C3.2, LED1.GND, R3.1, WEMOS1.GND
- removed net N$7: 4.2V_REGULATOR.EN, 4.2V_REGULATOR.VIN, C4.1, L2.1, TP4056.OUT+
- removed net TOGGLE_SWITCH: TOGGLE_SWITCH.O, WEMOS1.D7
- new net +5V: 5V_REGULATOR.VOUT, C1.1, C2.1, R2.2, SWITCH.P, WEMOS1.5V
- new net GND: 4.2V_REGULATOR.GND, 4.2V_REGULATOR.MODE, 5V_REGULATOR.GND, 5V_REGULATOR.MODE, C2.2, C3.2, C4.2, C5.1, LED1.GND, R3.1, R5.1, SIM800L.GND, TP4056.OUT-, WEMOS1.GND
- new net V+: 4.2V_REGULATOR.EN, 4.2V_REGULATOR.VIN, 5V_REGULATOR.EN, 5V_REGULATOR.VIN, C3.1, C4.1, L1.1, L2.1, TP4056.OUT+
- new net VCC: 4.2V_REGULATOR.VOUT, C5.2, R4.2
- net N$12: now also SIM800L.RST, SIM800L.VCC; no longer 4.2V_REGULATOR.GND, 4.2V_REGULATOR.MODE, C4.2, C5.1, R5.1, SIM800L.GND, TP4056.OUT-
- net N$13: now also SWITCH.O, WEMOS1.D7; no longer 4.2V_REGULATOR.VOUT, C5.2, R4.2, SIM800L.VCC
Other:
- moved on the sheet: 4.2V_REGULATOR, 5V_REGULATOR, BATTERIE-1, BATTERIE-2, C1, C2, C3, C4, C5, L1, L2, R1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

Commit message: Board finished
Parts:
- C5: value 10uF -> 33uF
- R2: value 100kΩ -> 732kΩ
- R3, R5: value 732kΩ -> 100kΩ
- R4: value 100kΩ -> 604kΩ
Connections:
- removed net N$12: SIM800L.RST, SIM800L.VCC
- net VCC: now also SIM800L.VCC
Other:
- moved on the sheet: 4.2V_REGULATOR, 5V_REGULATOR, BATTERIE-1, BATTERIE-2, C1, C2, C3, C4, C5, L1, L2, R1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
